File: PCB_REVC/PCB.kicad_pcb (KiCad board)
At the start: 4 copper layers, 83 x 45.5 mm, 87 parts, among them J1 AudioJack3, J10 Conn_01x01_Pin, J11 Conn_01x01_Pin, J12 Conn_01x01_Pin, J13 Conn_01x01_Pin, J14 Conn_01x01_Pin, J15 Conn_01x08_Socket, J16 Conn_01x01_Pin, J17 Conn_01x01_Pin, J18 Conn_01x01_Pin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

Commit message: Adaugat ultima iteratie a PCB-ului si realizat interfata grafica
Parts:
- added G***: LOGO, footprints:Logo, F.Cu at (170.0, 108.0)
- C10, C16, C17, C19, C20, C6: value 100n -> 0.1u
- C11: value 220n -> 0.22u
- C12, C13, C15: value 120n -> 0.1u
- C14: value 4.7n -> 4700p
- C18: footprint Capacitor_SMD:C_1206_3216Metric_Pad1.33x1.80mm_HandSolder -> Capacitor_Tantalum_SMD:CP_EIA-3216-18_Kemet-A_HandSolder
- C21: value 100n -> 1u; footprint Capacitor_SMD:C_1206_3216Metric_Pad1.33x1.80mm_HandSolder -> Capacitor_Tantalum_SMD:CP_EIA-3216-18_Kemet-A_HandSolder
- C5: value 1n -> 1000p
- D1, D2, D3, D4, D5: value 3V3 -> 3V6
- R15: value 634k -> 620k
- turned C18 to -90 degrees
Routing:
- net Vcc: track 55.0 -> 52.8 mm
Other:
- board text added: "*"
- board text added: "CardioMed Rev B Bota Andrei-Daniel"
