File: PCB_REVC/PCB.kicad_sch (KiCad schematic)
At the start: 87 parts, among them J1 AudioJack3, J10 Conn_01x01_Pin, J11 Conn_01x01_Pin, J12 Conn_01x01_Pin, J13 Conn_01x01_Pin, J14 Conn_01x01_Pin, J15 Conn_01x08_Socket, J16 Conn_01x01_Pin, J17 Conn_01x01_Pin, J18 Conn_01x01_Pin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

Commit message: Adaugat ultima iteratie a PCB-ului si realizat interfata grafica
Parts:
- C1, C2, C3: Field5 https://ro.farnell.com/kemet/c0603c105k4ractu/cap-1-f-16v-1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 -> https://ro.farnell.com/multicomp-pro/1206b105j250cp/cap-1uf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
- C10, C6: value 100n -> 0.1u; Field5 https://ro.farnell.com/samsung-electro-mechanics/cl10b104kb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 -> https://ro.farnell.com/avx/12065c104jat2a/cap-0-1-f-50v-5-x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
- C11: value 220n -> 0.22u; Field5 https://ro.farnell.com/yageo/cc0603kpx7r8bb224/cap-0-22uf-2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 -> https://ro.farnell.com/avx/12065c224jat2a/cap-0-22-f-50v-5-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
- C12, C13, C15: value 120n -> 0.1u; Field5 https://ro.farnell.com/yageo/cc0603krx7r6bb124/capacitor-0-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 -> https://ro.farnell.com/avx/12065c104jat2a/cap-0-1-f-50v-5-x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
- C14: value 4.7n -> 4700p; Field5 https://ro.farnell.com/multicomp-pro/mc0603b472k500ct/cap-4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 -> https://ro.farnell.com/kemet/c1206c472j5ractu/cap-4700pf-50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
- C16, C17, C19, C20: value 100n -> 0.1u; Field5 https://ro.farnell.com/multicomp-pro/mc0603b472k500ct/cap-4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 -> https://ro.farnell.com/avx/12065c104jat2a/cap-0-1-f-50v-5-x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
- C18: footprint Capacitor_SMD:C_1206_3216Metric_Pad1.33x1.80mm_HandSolder -> Capacitor_Tantalum_SMD:CP_EIA-3216-18_Kemet-A_HandSolder; Field5 https://ro.farnell.com/multicomp-pro/mc0603b472k500ct/cap-4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 -> https://ro.farnell.com/kemet/t491a105k025at/cap-1-f-25v-10-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
- C21: value 100n -> 1u; footprint Capacitor_SMD:C_1206_3216Metric_Pad1.33x1.80mm_HandSolder -> Capacitor_Tantalum_SMD:CP_EIA-3216-18_Kemet-A_HandSolder; Field5 https://ro.farnell.com/multicomp-pro/mc0603b472k500ct/cap-4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 -> https://ro.farnell.com/kemet/t491a105k025at/cap-1-f-25v-10-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
- C4: Field5 https://ro.farnell.com/samsung-electro-mechanics/cl10b104kb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 -> https://ro.farnell.com/avx/12065c104jat2a/cap-0-1-f-50v-5-x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
- C5: value 1n -> 1000p; Field5 https://ro.farnell.com/kemet/c0603c102f4hactu/cap-1000pf-16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 -> https://ro.farnell.com/multicomp-pro/1206n102j500ct/cap-100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
- C7, C8, C9: Field5 https://ro.farnell.com/murata/grm188z71a106ka73d/cap-10uf-1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 -> https://ro.farnell.com/samsung-electro-mechanics/cl31b106ka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
- D1, D2, D3, D4, D5: Field5 https://ro.farnell.com/multicomp-pro/bzx84c3v3/zener-diode-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 -> https://ro.farnell.com/diodes-inc/bzx84c3v6/diode-zener-3-6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
- D6: Field5 https://ro.farnell.com/qt-brightek/qblp631-ag1/led-green-08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 -> https://ro.farnell.com/qt-brightek/qblp650-o/led-orange-120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
- J10, J11, J12, J13, J14, J16, J17, J18, J19, J20, J21, J22, J24, J3, J4, J5, J6, J7, J8, J9: Field5 https://ro.farnell.com/amphenol-communications-solutions/10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 -> https://ro.farnell.com/harwin/m20-9774046/connector-header-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
- J15, J2: Field5 (none) -> https://ro.farnell.com/harwin/m20-7820842/connector-rcpt-8p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
- R1, R2: Field5 https://ro.farnell.com/multicomp-pro/wf06u1003btl/res-100k-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 -> https://ro.farnell.com/yageo/rt1206brd07100kl/res-100k-0-1-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
- R10: Field5 https://ro.farnell.com/yageo/re0603dr-071ml/res-1m-0-5-0-1w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 -> https://ro.farnell.com/koa/rn73r2bttd1004b25/res-1m-0-25w-m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
- R11: Field5 https://ro.farnell.com/yageo/rt0603brd07316kl/res-316k-0-1-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 -> https://ro.farnell.com/yageo/rc1206fr-07316kl/res-316k-1-0-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
- R12: Field5 https://ro.farnell.com/panasonic/era3aeb912v/res-9k1-0-1-0-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 -> https://ro.farnell.com/multicomp-pro/mcwr12x9101ftl/res-9k1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
- R13, R19, R31: Field5 https://ro.farnell.com/multicomp-pro/mcwr06x1001ftl/res-1k-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 -> https://ro.farnell.com/multicomp-pro/wr12x1001ftl/res-1k-1-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
- R14: Field5 https://ro.farnell.com/te-connectivity/cpf0603b158ke1/res-1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 -> https://ro.farnell.com/panasonic/erj8enf1583v/res-158k-1-0-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
- R15: value 634k -> 620k; Field5 https://ro.farnell.com/multicomp-pro/wr06x6343ftl/res-634k-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 -> https://ro.farnell.com/vishay/crcw1206620kfkea/res-620k-1-0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
- R16, R17: Field5 https://ro.farnell.com/multicomp-pro/mcwf06r3162btl/res-31k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 -> https://ro.farnell.com/panasonic/era8aeb3162v/res-31k6-0-1-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
- R18: Field5 https://ro.farnell.com/panasonic/era3aeb1542v/res-15k4-0603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 -> https://ro.farnell.com/vishay/crcw120615k4fkea/res-15k4-1-0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
- R20, R4, R6: Field5 https://ro.farnell.com/multicomp-pro/wf06u1002btl/res-10k-0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 -> https://ro.farnell.com/yageo/rt1206brd0710kl/res-10k-0-1-0-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
- R21: Field5 https://ro.farnell.com/yageo/rt0603brd073k92l/res-3k92-0-1-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 -> https://ro.farnell.com/yageo/rc1206fr-073k92l/res-3k92-1-0-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
- R22: Field5 https://ro.farnell.com/yageo/rt0603brd0723k7l/res-23k7-0-1-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 -> https://ro.farnell.com/yageo/rc1206fr-0723k7l/res-23k7-1-0-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
- R23: Field5 https://ro.farnell.com/yageo/rt0603brd077k15l/res-7k15-0-1w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 -> https://ro.farnell.com/yageo/rc1206fr-077k15l/res-7k15-1-0-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
- R24: Field5 https://ro.farnell.com/panasonic/era3aeb2871v/res-2k87-0603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 -> https://ro.farnell.com/yageo/rc1206fr-072k87l/res-2k87-1-0-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
- R25: Field5 https://ro.farnell.com/panasonic/era3aeb8661v/res-8k66-0-1-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 -> https://ro.farnell.com/yageo/rc1206fr-078k66l/res-8k66-1-0-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
- R26: Field5 https://ro.farnell.com/panasonic/era3aeb2743v/res-274k-0-1-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 -> https://ro.farnell.com/yageo/rc1206fr-07274kl/res-274k-1-0-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
- R27: Field5 https://ro.farnell.com/panasonic/era3aeb3011v/res-3k01-0-1-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 -> https://ro.farnell.com/bourns/cr1206-fx-3011elf/res-3k01-1-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
- R28: Field5 https://ro.farnell.com/yageo/rt0603brd076k81l/res-6k81-0-1-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 -> https://ro.farnell.com/yageo/rc1206fr-076k81l/res-6k81-1-0-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
- R3, R5: Field5 https://ro.farnell.com/multicomp-pro/wf06u2002btl/res-20k-0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 -> https://ro.farnell.com/multicomp-pro/mcwr12x2002ftl/res-20k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
- R7, R8, R9: Field5 https://ro.farnell.com/vishay/crcw060310m0dheap/res-10m-0-5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 -> https://ro.farnell.com/vishay/crcw120610m0dheap/res-aec-q20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

Commit message: Adaugat PanTompkins detectie
Parts:
- C1, C11, C2, C3, D6: Price (none) -> 0,3388 lei
- C10, C12, C13, C14, C15, C16, C17, C19, C20, C4, C5, C6: Price (none) -> 0,2541 lei
- C18, C21: Price (none) -> 0,6776 lei
- C7, C8, C9: Price (none) -> 0,3509 lei
- D1, D2, D3, D4, D5: Price (none) -> 0,2662 lei
- D7, D8: Price (none) -> 0,7744 lei
- J1: Price (none) -> 3,1097 lei
- J10, J11, J12, J13, J14, J16, J17, J18, J19, J20, J21, J22, J24, J3, J4, J5, J6, J7, J8, J9: Price (none) -> 5,203 lei
- J15, J2: Price (none) -> 5,0699 lei
- R1, R2: Price (none) -> 0,7018 lei
- R10: Price (none) -> 0,7502 lei
- R11, R21, R23, R24, R25, R26, R28: Price (none) -> 0,0726 lei
- R12, R13, R19, R3, R31, R5: Price (none) -> 0,0484 lei
- R14: Price (none) -> 0,1815 lei
- R15, R18: Price (none) -> 0,121 lei
- R16, R17: Price (none) -> 1,2221 lei
- R20, R4, R6: Price (none) -> 0,6655 lei
- R22, R27: Price (none) -> 0,0605 lei
- R7, R8, R9: Price (none) -> 0,4961 lei
- U1: Field5 (none) -> https://ro.farnell.com/analog-devices/adp151aujz-3-3-r7/ldo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; Price (none) -> 4,6464 lei
- U2: Field5 (none) -> https://ro.farnell.com/analog-devices/max41400atb-t/instrum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; Price (none) -> 11,3861 lei
- U3, U6: Field5 (none) -> https://ro.farnell.com/analog-devices/ad8534arz/op-amp-3mhz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; Price (none) -> 6,897 lei
- U4: Field5 (none) -> https://ro.farnell.com/analog-devices/ad7124-4bruz/adc-24bi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; Price (none) -> 51,3887 lei
- U5: Field5 (none) -> https://www.alibaba.com/product-detail/ESP32-C3-Super-Mini-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; Price None -> 9,40 RON
